File: UV360/_autosave-mcu.kicad_sch (KiCad schematic)
At the start: 2 parts, among them U1 STM32_BlackPill

Commit message: mcu
Connections:
- net PA8 renamed A8/GPIO_IN
- net PA9 renamed A9/GPIO_IN
- net PB12 renamed B12/GPIO_IN
- net PB13 renamed B13/GPIO_IN
- net PB14 renamed B14/GPIO_IN
- net PB15 renamed B15/GPIO_IN
- net PB5/GPIO_IN renamed PB5
- net PB8/GPIO_IN renamed PB8
- net PB9/GPIO_IN renamed PB9
- net PC13/GPIO_IN renamed PC13
- net PC14/GPIO_IN renamed PC14
- net PC15/GPIO_IN renamed PC15
- no-connect marks 18 -> 22
Changed lines of the file:
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@@
-	)
-	(no_connect
-		(at 151.13 68.58)
 	)
 	(no_connect
@@
 	)
 	(no_connect
+		(at 151.13 104.14)
+	)
+	(no_connect
 		(at 171.45 66.04)
 	)
@@
 	)
 	(no_connect
-		(at 151.13 66.04)
-	)
-	(no_connect
-		(at 151.13 71.12)
-	)
-	(no_connect
-		(at 151.13 73.66)
+		(at 151.13 91.44)
+	)
+	(no_connect
+		(at 171.45 106.68)
+	)
+	(no_connect
+		(at 151.13 93.98)
 	)
 	(no_connect
@@
 	)
 	(no_connect
-		(at 151.13 76.2)
+		(at 171.45 109.22)
+	)
+	(no_connect
+		(at 171.45 104.14)
+	)
+	(no_connect
+		(at 151.13 101.6)
 	)
 	(no_connect
 		(at 171.45 91.44)
 	)
+	(no_connect
+		(at 151.13 86.36)
+	)
+	(no_connect
+		(at 151.13 88.9)
+	)
 	(wire
 		(pts
@@
 	(wire
 		(pts
+			(xy 135.89 73.66) (xy 151.13 73.66)
+		)
+		(stroke
+			(width 0)
+			(type default)
+		)
+	)
+	(wire
+		(pts
 			(xy 171.45 83.82) (xy 182.88 83.82)
 		)
@@
 	(wire
 		(pts
+			(xy 135.89 76.2) (xy 151.13 76.2)
+		)
+		(stroke
+			(width 0)
+			(type default)
+		)
+	)
+	(wire
+		(pts
 			(xy 135.89 99.06) (xy 151.13 99.06)
 		)
@@
 	(wire
 		(pts
+			(xy 135.89 63.5) (xy 151.13 63.5)
+		)
+		(stroke
+			(width 0)
+			(type default)
+		)
+	)
+	(wire
+		(pts
 			(xy 142.24 109.22) (xy 151.13 109.22)
 		)
@@
 	(wire
 		(pts
+			(xy 135.89 66.04) (xy 151.13 66.04)
+		)
+		(stroke
+			(width 0)
+			(type default)
+		)
+	)
+	(wire
+		(pts
 			(xy 171.45 96.52) (xy 182.88 96.52)
 		)
@@
 	(wire
 		(pts
+			(xy 135.89 71.12) (xy 151.13 71.12)
+		)
+		(stroke
+			(width 0)
+			(type default)
+		)
+	)
+	(wire
+		(pts
 			(xy 171.45 99.06) (xy 182.88 99.06)
+		)
+		(stroke
+			(width 0)
+			(type default)
+		)
+	)
+	(wire
+		(pts
+			(xy 135.89 68.58) (xy 151.13 68.58)
 		)
 		(stroke
@@
 		)
 	)
-	(label "PA9"
-		(at 151.13 76.2 180)
-		(effects
-			(font
-				(size 1.27 1.27)
-			)
-			(justify right bottom)
-		)
-	)
 	(label "PA6"
 		(at 171.45 83.82 0)
@@
 		)
 	)
-	(label "PC13"
-		(at 92.71 95.25 0)
-		(effects
-			(font
-				(size 1.27 1.27)
-			)
-			(justify left bottom)
-		)
-	)
 	(label "PA11"
 		(at 151.13 81.28 180)
@@
 		)
 	)
-	(label "PB5"
-		(at 92.71 85.09 0)
-		(effects
-			(font
-				(size 1.27 1.27)
-			)
-			(justify left bottom)
-		)
-	)
 	(label "PB9"
 		(at 151.13 104.14 180)
@@
 		)
 	)
-	(label "PB12"
-		(at 151.13 63.5 180)
-		(effects
-			(font
-				(size 1.27 1.27)
-			)
-			(justify right bottom)
-		)
-	)
-	(label "PB8"
-		(at 92.71 87.63 0)
-		(effects
-			(font
-				(size 1.27 1.27)
-			)
-			(justify left bottom)
-		)
-	)
-	(label "PB9"
-		(at 92.71 90.17 0)
-		(effects
-			(font
-				(size 1.27 1.27)
-			)
-			(justify left bottom)
-		)
-	)
-	(label "PC15"
-		(at 92.71 100.33 0)
-		(effects
-			(font
-				(size 1.27 1.27)
-			)
-			(justify left bottom)
-		)
-	)
 	(label "PC14"
 		(at 171.45 106.68 0)
@@
 		)
 	)
-	(label "PA8"
-		(at 151.13 73.66 180)
-		(effects
-			(font
-				(size 1.27 1.27)
-			)
-			(justify right bottom)
-		)
-	)
-	(label "PB13"
-		(at 151.13 66.04 180)
-		(effects
-			(font
-				(size 1.27 1.27)
-			)
-			(justify right bottom)
-		)
-	)
-	(label "PC14"
-		(at 92.71 97.79 0)
-		(effects
-			(font
-				(size 1.27 1.27)
-			)
-			(justify left bottom)
-		)
-	)
 	(label "PB0"
 		(at 171.45 78.74 0)
@@
 		)
 	)
-	(label "PB14"
-		(at 151.13 68.58 180)
-		(effects
-			(font
-				(size 1.27 1.27)
-			)
-			(justify right bottom)
-		)
-	)
 	(label "PC13"
 		(at 171.45 109.22 0)
@@
 		)
 	)
-	(label "PB15"
-		(at 151.13 71.12 180)
-		(effects
-			(font
-				(size 1.27 1.27)
-			)
-			(justify right bottom)
-		)
-	)
 	(label "PA15"
 		(at 151.13 86.36 180)
@@
 		)
 	)
-	(hierarchical_label "PC13{slash}GPIO_IN"
-		(shape input)
-		(at 92.71 95.25 180)
-		(effects
-			(font
-				(size 1.27 1.27)
-			)
-			(justify right)
-		)
-	)
 	(hierarchical_label "PB0{slash}SWO"
 		(shape input)
@@
 		)
 	)
-	(hierarchical_label "PB5{slash}GPIO_IN"
-		(shape input)
-		(at 92.71 85.09 180)
-		(effects
-			(font
-				(size 1.27 1.27)
-			)
-			(justify right)
-		)
-	)
 	(hierarchical_label "GND"
 		(shape input)
@@
 		)
 	)
+	(hierarchical_label "B14{slash}GPIO_IN"
+		(shape input)
+		(at 135.89 68.58 180)
+		(effects
+			(font
+				(size 1.27 1.27)
+			)
+			(justify right)
+		)
+	)
+	(hierarchical_label "B15{slash}GPIO_IN"
+		(shape input)
+		(at 135.89 71.12 180)
+		(effects
+			(font
+				(size 1.27 1.27)
+			)
+			(justify right)
+		)
+	)
 	(hierarchical_label "PB7{slash}I2C_SDA1"
 		(shape input)
@@
 		)
 	)
-	(hierarchical_label "PB8{slash}GPIO_IN"
-		(shape input)
-		(at 92.71 87.63 180)
-		(effects
-			(font
-				(size 1.27 1.27)
-			)
-			(justify right)
-		)
-	)
-	(hierarchical_label "PC14{slash}GPIO_IN"
-		(shape input)
-		(at 92.71 97.79 180)
-		(effects
-			(font
-				(size 1.27 1.27)
-			)
-			(justify right)
-		)
-	)
-	(hierarchical_label "PB3{slash}GPIO_IN"
-		(shape input)
-		(at 110.49 69.85 180)
-		(effects
-			(font
-				(size 1.27 1.27)
-			)
-			(justify right)
-		)
-	)
-	(hierarchical_label "PB9{slash}GPIO_IN"
-		(shape input)
-		(at 92.71 90.17 180)
-		(effects
-			(font
-				(size 1.27 1.27)
-			)
-			(justify right)
-		)
-	)
 	(hierarchical_label "PA0{slash}ENCODER_TIM2_CH1"
 		(shape input)
@@
 		)
 	)
-	(hierarchical_label "PC15{slash}GPIO_IN"
-		(shape input)
-		(at 92.71 100.33 180)
+	(hierarchical_label "B12{slash}GPIO_IN"
+		(shape input)
+		(at 135.89 63.5 180)
 		(effects
 			(font
@@
 		)
 	)
+	(hierarchical_label "A9{slash}GPIO_IN"
+		(shape input)
+		(at 135.89 76.2 180)
+		(effects
+			(font
+				(size 1.27 1.27)
+			)
+			(justify right)
+		)
+	)
 	(hierarchical_label "5V"
 		(shape input)
@@
 		)
 	)
+	(hierarchical_label "A8{slash}GPIO_IN"
+		(shape input)
+		(at 135.89 73.66 180)
+		(effects
+			(font
+				(size 1.27 1.27)
+			)
+			(justify right)
+		)
+	)
 	(hierarchical_label "PA6{slash}EEPROM_SPI1_MISO"
 		(shape input)
@@
 		)
 	)
+	(hierarchical_label "B13{slash}GPIO_IN"
+		(shape input)
+		(at 135.89 66.04 180)
+		(effects
+			(font
+				(size 1.27 1.27)
+			)
+			(justify right)
+		)
+	)
