File: UV360/UV360.kicad_sch (KiCad schematic)
At the start: 5 parts

Commit message: mcu
Connections:
- no-connect marks 0 -> 4
Other:
- sheet MCU ports: added A8/GPIO_IN, A9/GPIO_IN, B12/GPIO_IN, B13/GPIO_IN, B14/GPIO_IN, B15/GPIO_IN, PB0/SWO; removed PB3/GPIO_IN, PB5/GPIO_IN, PB8/GPIO_IN, PB9/GPIO_IN, PC13/GPIO_IN, PC14/GPIO_IN, PC15/GPIO_IN
- moved on the sheet: H1, H2, H3, H4
Changed lines of the file:
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@@
 	(generator_version "9.0")
 	(paper "A4")
+	(no_connect
+		(at 187.96 105.41)
+	)
+	(no_connect
+		(at 187.96 110.49)
+	)
+	(no_connect
+		(at 187.96 107.95)
+	)
+	(no_connect
+		(at 187.96 102.87)
+	)
+	(wire
+		(pts
+			(xy 86.36 74.93) (xy 130.81 74.93)
+		)
+		(stroke
+			(width 0)
+			(type default)
+		)
+	)
+	(wire
+		(pts
+			(xy 187.96 77.47) (xy 213.36 77.47)
+		)
+		(stroke
+			(width 0)
+			(type default)
+		)
+	)
+	(wire
+		(pts
+			(xy 86.36 88.9) (xy 130.81 88.9)
+		)
+		(stroke
+			(width 0)
+			(type default)
+		)
+	)
+	(wire
+		(pts
+			(xy 86.36 77.47) (xy 130.81 77.47)
+		)
+		(stroke
+			(width 0)
+			(type default)
+		)
+	)
+	(wire
+		(pts
+			(xy 187.96 80.01) (xy 213.36 80.01)
+		)
+		(stroke
+			(width 0)
+			(type default)
+		)
+	)
 	(wire
 		(pts
@@
 	(wire
 		(pts
-			(xy 245.11 60.96) (xy 251.46 60.96)
+			(xy 86.36 110.49) (xy 130.81 110.49)
 		)
 		(stroke
@@
 		)
 	)
+	(wire
+		(pts
+			(xy 245.11 60.96) (xy 251.46 60.96)
+		)
+		(stroke
+			(width 0)
+			(type default)
+		)
+	)
+	(wire
+		(pts
+			(xy 86.36 107.95) (xy 130.81 107.95)
+		)
+		(stroke
+			(width 0)
+			(type default)
+		)
+	)
+	(wire
+		(pts
+			(xy 86.36 86.36) (xy 130.81 86.36)
+		)
+		(stroke
+			(width 0)
+			(type default)
+		)
+	)
+	(wire
+		(pts
+			(xy 86.36 105.41) (xy 130.81 105.41)
+		)
+		(stroke
+			(width 0)
+			(type default)
+		)
+	)
+	(wire
+		(pts
+			(xy 86.36 91.44) (xy 130.81 91.44)
+		)
+		(stroke
+			(width 0)
+			(type default)
+		)
+	)
+	(wire
+		(pts
+			(xy 86.36 72.39) (xy 130.81 72.39)
+		)
+		(stroke
+			(width 0)
+			(type default)
+		)
+	)
 	(symbol
 		(lib_id "Mechanical:MountingHole")
-		(at 157.48 143.51 0)
+		(at 170.18 153.67 0)
 		(unit 1)
 		(exclude_from_sim no)
@@
 		(fields_autoplaced yes)
 		(property "Reference" "H4"
-			(at 160.02 142.2399 0)
+			(at 172.72 152.3999 0)
 			(effects
 				(font
@@
 		)
 		(property "Value" "MountingHole"
-			(at 160.02 144.7799 0)
+			(at 172.72 154.9399 0)
 			(effects
 				(font
@@
 		)
 		(property "Footprint" "MountingHole:MountingHole_4.3mm_M4"
-			(at 157.48 143.51 0)
+			(at 170.18 153.67 0)
 			(effects
 				(font
@@
 		)
 		(property "Datasheet" "~"
-			(at 157.48 143.51 0)
+			(at 170.18 153.67 0)
 			(effects
 				(font
@@
 		)
 		(property "Description" "Mounting Hole without connection"
-			(at 157.48 143.51 0)
+			(at 170.18 153.67 0)
 			(effects
 				(font
@@
 	(symbol
 		(lib_id "Mechanical:MountingHole")
-		(at 133.35 143.51 0)
+		(at 146.05 153.67 0)
 		(unit 1)
 		(exclude_from_sim no)
@@
 		(fields_autoplaced yes)
 		(property "Reference" "H3"
-			(at 135.89 142.2399 0)
+			(at 148.59 152.3999 0)
 			(effects
 				(font
@@
 		)
 		(property "Value" "MountingHole"
-			(at 135.89 144.7799 0)
+			(at 148.59 154.9399 0)
 			(effects
 				(font
@@
 		)
 		(property "Footprint" "MountingHole:MountingHole_4.3mm_M4"
-			(at 133.35 143.51 0)
+			(at 146.05 153.67 0)
 			(effects
 				(font
@@
 		)
 		(property "Datasheet" "~"
-			(at 133.35 143.51 0)
+			(at 146.05 153.67 0)
 			(effects
 				(font
@@
 		)
 		(property "Description" "Mounting Hole without connection"
-			(at 133.35 143.51 0)
+			(at 146.05 153.67 0)
 			(effects
 				(font
@@
 	(symbol
 		(lib_id "Mechanical:MountingHole")
-		(at 157.48 135.89 0)
+		(at 170.18 146.05 0)
 		(unit 1)
 		(exclude_from_sim no)
@@
 		(fields_autoplaced yes)
 		(property "Reference" "H2"
-			(at 160.02 134.6199 0)
+			(at 172.72 144.7799 0)
 			(effects
 				(font
@@
 		)
 		(property "Value" "MountingHole"
-			(at 160.02 137.1599 0)
+			(at 172.72 147.3199 0)
 			(effects
 				(font
@@
 		)
 		(property "Footprint" "MountingHole:MountingHole_4.3mm_M4"
-			(at 157.48 135.89 0)
+			(at 170.18 146.05 0)
 			(effects
 				(font
@@
 		)
 		(property "Datasheet" "~"
-			(at 157.48 135.89 0)
+			(at 170.18 146.05 0)
 			(effects
 				(font
@@
 		)
 		(property "Description" "Mounting Hole without connection"
-			(at 157.48 135.89 0)
+			(at 170.18 146.05 0)
 			(effects
 				(font
@@
 	(symbol
 		(lib_id "Mechanical:MountingHole")
-		(at 133.35 135.89 0)
+		(at 146.05 146.05 0)
 		(unit 1)
 		(exclude_from_sim no)
@@
 		(fields_autoplaced yes)
 		(property "Reference" "H1"
-			(at 135.89 134.6199 0)
+			(at 148.59 144.7799 0)
 			(effects
 				(font
@@
 		)
 		(property "Value" "MountingHole"
-			(at 135.89 137.1599 0)
+			(at 148.59 147.3199 0)
 			(effects
 				(font
@@
 		)
 		(property "Footprint" "MountingHole:MountingHole_4.3mm_M4"
-			(at 133.35 135.89 0)
+			(at 146.05 146.05 0)
 			(effects
 				(font
@@
 		)
 		(property "Datasheet" "~"
-			(at 133.35 135.89 0)
+			(at 146.05 146.05 0)
 			(effects
 				(font
@@
 		)
 		(property "Description" "Mounting Hole without connection"
-			(at 133.35 135.89 0)
+			(at 146.05 146.05 0)
 			(effects
 				(font
@@
 		)
 		(pin "CLK" input
-			(at 86.36 110.49 0)
+			(at 86.36 107.95 0)
 			(effects
 				(font
@@
 		)
 		(pin "DT" input
-			(at 86.36 107.95 0)
+			(at 86.36 105.41 0)
 			(effects
 				(font
@@
 		)
 		(pin "SW" input
-			(at 86.36 105.41 0)
+			(at 86.36 110.49 0)
 			(effects
 				(font
@@
 			)
 		)
-		(pin "PB3{slash}GPIO_IN" input
-			(at 130.81 68.58 180)
-			(effects
-				(font
-					(size 1.27 1.27)
-				)
-				(justify left)
-			)
-		)
-		(pin "PB5{slash}GPIO_IN" input
-			(at 130.81 71.12 180)
-			(effects
-				(font
-					(size 1.27 1.27)
-				)
-				(justify left)
-			)
-		)
 		(pin "PB6{slash}I2C_SCL1" input
-			(at 187.96 82.55 0)
+			(at 187.96 77.47 0)
 			(effects
 				(font
@@
 		)
 		(pin "PB7{slash}I2C_SDA1" input
-			(at 187.96 85.09 0)
-			(effects
-				(font
-					(size 1.27 1.27)
-				)
-				(justify right)
-			)
-		)
-		(pin "PB8{slash}GPIO_IN" input
-			(at 130.81 73.66 180)
-			(effects
-				(font
-					(size 1.27 1.27)
-				)
-				(justify left)
-			)
-		)
-		(pin "PB9{slash}GPIO_IN" input
-			(at 130.81 76.2 180)
-			(effects
-				(font
-					(size 1.27 1.27)
-				)
-				(justify left)
-			)
-		)
-		(pin "PC13{slash}GPIO_IN" input
-			(at 130.81 87.63 180)
-			(effects
-				(font
-					(size 1.27 1.27)
-				)
-				(justify left)
-			)
-		)
-		(pin "PC14{slash}GPIO_IN" input
-			(at 130.81 90.17 180)
-			(effects
-				(font
-					(size 1.27 1.27)
-				)
-				(justify left)
-			)
-		)
-		(pin "PC15{slash}GPIO_IN" input
-			(at 130.81 92.71 180)
-			(effects
-				(font
+			(at 187.96 80.01 0)
+			(effects
+				(font
+					(size 1.27 1.27)
+				)
+				(justify right)
+			)
+		)
+		(pin "A8{slash}GPIO_IN" input
+			(at 130.81 86.36 180)
+			(effects
+				(font
+					(size 1.27 1.27)
+				)
+				(justify left)
+			)
+		)
+		(pin "A9{slash}GPIO_IN" input
+			(at 130.81 88.9 180)
+			(effects
+				(font
+					(size 1.27 1.27)
+				)
+				(justify left)
+			)
+		)
+		(pin "B12{slash}GPIO_IN" input
+			(at 130.81 72.39 180)
+			(effects
+				(font
+					(size 1.27 1.27)
+				)
+				(justify left)
+			)
+		)
+		(pin "B13{slash}GPIO_IN" input
+			(at 130.81 74.93 180)
+			(effects
+				(font
+					(size 1.27 1.27)
+				)
+				(justify left)
+			)
+		)
+		(pin "B14{slash}GPIO_IN" input
+			(at 130.81 77.47 180)
+			(effects
+				(font
+					(size 1.27 1.27)
+				)
+				(justify left)
+			)
+		)
+		(pin "B15{slash}GPIO_IN" input
+			(at 130.81 91.44 180)
+			(effects
+				(font
+					(size 1.27 1.27)
+				)
+				(justify left)
+			)
+		)
+		(pin "PB0{slash}SWO" input
+			(at 130.81 99.06 180)
+			(effects
+				(font
