File: UV360/UV360.kicad_sch (KiCad schematic)
At the start: 5 parts

Commit message: PIR
Other:
- sheet MCU ports: added MCU-3.3V, MCU-3.3V-GND; removed none
- sheet PIR SENSORS ports: added +5V, GND-5V, MCU-3.3V, MCU-3.3V-GND; removed none
- sheet Power Section ports: added 3.3V-BUCK, 3.3V_GND-BUCK; removed 3.3V, 3.3V_GND
