File: UV360/power_section.kicad_sch (KiCad schematic)
At the start: 21 parts, among them J17 12V-SW, J5 12V-IN, J6 12V-OUT, U2 L7805

Commit message: PIR Section
Parts:
- added D1: DF10M, Diode_THT:Diode_Bridge_DIP-4_W7.62mm_P5.08mm, symbol Diode_Bridge:DF10M
- J17: value 12V-SW -> 9V AC-SW
- J5: value 12V-IN -> 9V AC-IN
- R4: value 1k -> 2.2K
Connections:
- net 12V: now also D1.1 (+); no longer J17.1 (Pin_1)
- net 12V_GND: now also D1.2 (-); no longer J5.2 (Pin_2)
- new net AC1: D1.4, J17.1 (Pin_1)
- new net AC2: D1.3, J5.2 (Pin_2)
Other:
- note added: "9V AC IN FROM TRANSFORMER"
- note added: "OPTIONAL SWITCH"
- moved on the sheet: BC2, C11, C17, C18, C19, C20, C21, C22, C23, C24, C25, C26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

Commit message: PIR
Connections:
- net 3.3V renamed 3.3V-BUCK
- net 3.3V_GND renamed 3.3V_GND-BUCK
Changed lines of the file:
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@@
 		)
 	)
-	(hierarchical_label "3.3V"
+	(hierarchical_label "3.3V-BUCK"
 		(shape output)
 		(at 218.44 124.46 0)
@@
 		)
 	)
-	(hierarchical_label "3.3V_GND"
+	(hierarchical_label "3.3V_GND-BUCK"
 		(shape output)
 		(at 218.44 140.97 0)
