File: UV360/hlk_sensors.kicad_sch (KiCad schematic)
At the start: 0 parts

Commit message: PIR
Parts:
- added C2: 0.1uf, Capacitor_THT:C_Disc_D3.8mm_W2.6mm_P2.50mm, symbol Device:C_Small
- added J?: HLK_SERIAL, TerminalBlock_Phoenix:TerminalBlock_Phoenix_MKDS-1,5-6-5.08_1x06_P5.08mm_Horizontal, symbol Connector:Screw_Terminal_01x06
- added J?: HLK2 SERIAL, TerminalBlock_Phoenix:TerminalBlock_Phoenix_MKDS-1,5-3-5.08_1x03_P5.08mm_Horizontal, symbol Connector:Screw_Terminal_01x03
- added J?: HLK, TerminalBlock_Phoenix:TerminalBlock_Phoenix_MKDS-1,5-5-5.08_1x05_P5.08mm_Horizontal, symbol Connector:Screw_Terminal_01x05
- added J?: HLK1 SERIAL, TerminalBlock_Phoenix:TerminalBlock_Phoenix_MKDS-1,5-3-5.08_1x03_P5.08mm_Horizontal, symbol Connector:Screw_Terminal_01x03
- added J?: HLK3 SERIAL, TerminalBlock_Phoenix:TerminalBlock_Phoenix_MKDS-1,5-3-5.08_1x03_P5.08mm_Horizontal, symbol Connector:Screw_Terminal_01x03
Connections:
- new net 3.3V: C2.1, J?.2 (Pin_2)
- new net GND: C2.2, J?.1 (Pin_1), J?.3 (Pin_3), J?.3 (Pin_3), J?.3 (Pin_3)
- new net HLK ISOLATOR/HLK: J?.3 (Pin_3)
- new net HLK ISOLATOR1/HLK: J?.4 (Pin_4)
- new net HLK ISOLATOR2/HLK: J?.5 (Pin_5)
- new net HLK1_RX: J?.1 (Pin_1), J?.2 (Pin_2)
- new net HLK1_TX: J?.1 (Pin_1), J?.2 (Pin_2)
- new net HLK2_RX: J?.1 (Pin_1), J?.4 (Pin_4)
- new net HLK2_TX: J?.2 (Pin_2), J?.3 (Pin_3)
- new net HLK3_RX: J?.1 (Pin_1), J?.6 (Pin_6)
- new net HLK3_TX: J?.2 (Pin_2), J?.5 (Pin_5)
Other:
- added sheet HLK ISOLATOR (hlk isolator.kicad_sch)
- added sheet HLK ISOLATOR1 (hlk isolator.kicad_sch)
- added sheet HLK ISOLATOR2 (hlk isolator.kicad_sch)
