File: UV360/mcu.kicad_sch (KiCad schematic)
At the start: 2 parts, among them U1 STM32_BlackPill

Commit message: PIR Section
Connections:
- no-connect marks 22 -> 20
Changed lines of the file:
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@@
-	)
-	(no_connect
-		(at 171.45 76.2)
 	)
 	(no_connect
@@
 	)
 	(no_connect
-		(at 171.45 73.66)
-	)
-	(no_connect

Commit message: PIR
Connections:
- net MCU-3.3V: now reaches U1.38 (3V3)
- net MCU-3.3V-GND: now reaches U1.39 (G)
- no-connect marks 20 -> 18
Changed lines of the file:
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@@
-	)
-	(no_connect
-		(at 171.45 66.04)
 	)
 	(no_connect
@@
 	)
 	(no_connect
-		(at 171.45 68.58)
-	)
-	(no_connect
 		(at 171.45 111.76)
 	)
@@
 	(wire
 		(pts
+			(xy 171.45 68.58) (xy 182.88 68.58)
+		)
+		(stroke
+			(width 0)
+			(type default)
+		)
+	)
+	(wire
+		(pts
 			(xy 171.45 88.9) (xy 182.88 88.9)
 		)
@@
 		(pts
 			(xy 171.45 86.36) (xy 182.88 86.36)
+		)
+		(stroke
+			(width 0)
+			(type default)
+		)
+	)
+	(wire
+		(pts
+			(xy 171.45 66.04) (xy 182.88 66.04)
 		)
 		(stroke
@@
 		)
 	)
+	(hierarchical_label "MCU-3.3V-GND"
+		(shape output)
+		(at 182.88 66.04 0)
+		(effects
+			(font
+				(size 1.27 1.27)
+			)
+			(justify left)
+		)
+	)
 	(hierarchical_label "PA7{slash}EEPROM_SPI1_MOSI"
 		(shape input)
@@
 		(effects
 			(font
+				(size 1.27 1.27)
+			)
+			(justify left)
+		)
+	)
+	(hierarchical_label "MCU-3.3V"
+		(shape output)
+		(at 182.88 68.58 0)
+		(effects
+			(font
