File: UV360/pir_isolator.kicad_sch (KiCad schematic)
At the start: 11 parts, among them Q2 BC547, U5 PC817

Commit message: PIR Section
Parts:
- R11: value 1k -> 22k
Other:
- note added: "Panassonic EKMC1604113 PIR Sensor Maximum Operating Current - 170uA Output Current - 100ua Output voltage - Vdd - 0.5 Vdd - 3.3v"
Changed lines of the file:
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@@
 	(generator_version "9.0")
 	(paper "A4")
+	(text "Panassonic EKMC1604113 PIR Sensor\nMaximum Operating Current - 170uA\nOutput Current - 100ua\nOutput voltage - Vdd - 0.5\nVdd - 3.3v"
+		(exclude_from_sim no)
+		(at 50.038 96.266 0)
+		(effects
+			(font
+				(size 1.27 1.27)
+			)
+			(justify left)
+		)
+	)
 	(junction
 		(at 133.35 118.11)
@@
 	(wire
 		(pts
-			(xy 152.4 96.52) (xy 153.67 96.52)
+			(xy 152.4 96.52) (xy 161.29 96.52)
 		)
 		(stroke
@@
 	(hierarchical_label "PIR_mcu"
 		(shape input)
-		(at 153.67 96.52 0)
+		(at 161.29 96.52 0)
 		(effects
 			(font
@@
 		(on_board yes)
 		(dnp no)
-		(property "Reference" "C8"
+		(property "Reference" "C?"
 			(at 120.65 81.534 90)
 			(effects
@@
 					(unit 1)
 				)
+				(path "/f41306b9-7b2a-47ad-8a6e-226fbfa024ae/5235c0b2-ed00-4052-87b3-aafa4437d860/838d61aa-bfd3-43b0-96be-35c67846f33d"
+					(reference "C?")
+					(unit 1)
+				)
+				(path "/f41306b9-7b2a-47ad-8a6e-226fbfa024ae/5235c0b2-ed00-4052-87b3-aafa4437d860/fdd530e1-065e-4c92-a13d-ffa8fd694749"
+					(reference "C?")
+					(unit 1)
+				)
 			)
 		)
@@
 		(on_board yes)
 		(dnp no)
-		(property "Reference" "#PWR010"
+		(property "Reference" "#PWR?"
 			(at 152.4 81.28 0)
 			(effects
@@
 					(unit 1)
 				)
+				(path "/f41306b9-7b2a-47ad-8a6e-226fbfa024ae/5235c0b2-ed00-4052-87b3-aafa4437d860/838d61aa-bfd3-43b0-96be-35c67846f33d"
+					(reference "#PWR?")
+					(unit 1)
+				)
+				(path "/f41306b9-7b2a-47ad-8a6e-226fbfa024ae/5235c0b2-ed00-4052-87b3-aafa4437d860/fdd530e1-065e-4c92-a13d-ffa8fd694749"
+					(reference "#PWR?")
+					(unit 1)
+				)
 			)
 		)
@@
 		(on_board yes)
 		(dnp no)
-		(property "Reference" "C13"
+		(property "Reference" "C?"
 			(at 117.348 111.506 0)
 			(effects
@@
 					(unit 1)
 				)
+				(path "/f41306b9-7b2a-47ad-8a6e-226fbfa024ae/5235c0b2-ed00-4052-87b3-aafa4437d860/838d61aa-bfd3-43b0-96be-35c67846f33d"
+					(reference "C?")
+					(unit 1)
+				)
+				(path "/f41306b9-7b2a-47ad-8a6e-226fbfa024ae/5235c0b2-ed00-4052-87b3-aafa4437d860/fdd530e1-065e-4c92-a13d-ffa8fd694749"
+					(reference "C?")
+					(unit 1)
+				)
 			)
 		)
@@
 		(on_board yes)
 		(dnp no)
-		(property "Reference" "R12"
+		(property "Reference" "R?"
 			(at 126.492 114.3 90)
 			(effects
@@
 					(unit 1)
 				)
+				(path "/f41306b9-7b2a-47ad-8a6e-226fbfa024ae/5235c0b2-ed00-4052-87b3-aafa4437d860/838d61aa-bfd3-43b0-96be-35c67846f33d"
+					(reference "R?")
+					(unit 1)
+				)
+				(path "/f41306b9-7b2a-47ad-8a6e-226fbfa024ae/5235c0b2-ed00-4052-87b3-aafa4437d860/fdd530e1-065e-4c92-a13d-ffa8fd694749"
+					(reference "R?")
+					(unit 1)
+				)
 			)
 		)
@@
 		(on_board yes)
 		(dnp no)
-		(property "Reference" "R11"
+		(property "Reference" "R?"
 			(at 110.49 111.252 90)
 			(effects
@@
 			)
 		)
-		(property "Value" "1k"
+		(property "Value" "22k"
 			(at 110.49 107.188 90)
 			(effects
@@
 					(unit 1)
 				)
+				(path "/f41306b9-7b2a-47ad-8a6e-226fbfa024ae/5235c0b2-ed00-4052-87b3-aafa4437d860/838d61aa-bfd3-43b0-96be-35c67846f33d"
+					(reference "R?")
+					(unit 1)
+				)
+				(path "/f41306b9-7b2a-47ad-8a6e-226fbfa024ae/5235c0b2-ed00-4052-87b3-aafa4437d860/fdd530e1-065e-4c92-a13d-ffa8fd694749"
+					(reference "R?")
+					(unit 1)
+				)
 			)
 		)
@@
 		(on_board yes)
 		(dnp no)
-		(property "Reference" "R8"
+		(property "Reference" "R?"
 			(at 129.032 82.55 90)
 			(effects
@@
 					(unit 1)
 				)
+				(path "/f41306b9-7b2a-47ad-8a6e-226fbfa024ae/5235c0b2-ed00-4052-87b3-aafa4437d860/838d61aa-bfd3-43b0-96be-35c67846f33d"
+					(reference "R?")
+					(unit 1)
+				)
+				(path "/f41306b9-7b2a-47ad-8a6e-226fbfa024ae/5235c0b2-ed00-4052-87b3-aafa4437d860/fdd530e1-065e-4c92-a13d-ffa8fd694749"
+					(reference "R?")
+					(unit 1)
+				)
 			)
 		)
@@
 		(on_board yes)
 		(dnp no)
-		(property "Reference" "D3"
+		(property "Reference" "D?"
 			(at 128.778 91.44 90)
 			(effects
@@
 					(unit 1)
 				)
+				(path "/f41306b9-7b2a-47ad-8a6e-226fbfa024ae/5235c0b2-ed00-4052-87b3-aafa4437d860/838d61aa-bfd3-43b0-96be-35c67846f33d"
+					(reference "D?")
+					(unit 1)
+				)
+				(path "/f41306b9-7b2a-47ad-8a6e-226fbfa024ae/5235c0b2-ed00-4052-87b3-aafa4437d860/fdd530e1-065e-4c92-a13d-ffa8fd694749"
+					(reference "D?")
+					(unit 1)
+				)
 			)
 		)
@@
 		(on_board yes)
 		(dnp no)
-		(property "Reference" "#PWR013"
+		(property "Reference" "#PWR?"
 			(at 151.13 111.76 0)
 			(effects
@@
 					(unit 1)
 				)
+				(path "/f41306b9-7b2a-47ad-8a6e-226fbfa024ae/5235c0b2-ed00-4052-87b3-aafa4437d860/838d61aa-bfd3-43b0-96be-35c67846f33d"
+					(reference "#PWR?")
+					(unit 1)
+				)
+				(path "/f41306b9-7b2a-47ad-8a6e-226fbfa024ae/5235c0b2-ed00-4052-87b3-aafa4437d860/fdd530e1-065e-4c92-a13d-ffa8fd694749"
+					(reference "#PWR?")
+					(unit 1)
+				)
 			)
 		)
@@
 		(on_board yes)
 		(dnp no)
-		(property "Reference" "#PWR09"
+		(property "Reference" "#PWR?"
 			(at 133.35 81.28 0)
 			(effects
@@
 					(unit 1)
 				)
+				(path "/f41306b9-7b2a-47ad-8a6e-226fbfa024ae/5235c0b2-ed00-4052-87b3-aafa4437d860/838d61aa-bfd3-43b0-96be-35c67846f33d"
+					(reference "#PWR?")
+					(unit 1)
+				)
+				(path "/f41306b9-7b2a-47ad-8a6e-226fbfa024ae/5235c0b2-ed00-4052-87b3-aafa4437d860/fdd530e1-065e-4c92-a13d-ffa8fd694749"
+					(reference "#PWR?")
+					(unit 1)
+				)
 			)
 		)
@@
 		(on_board yes)
 		(dnp no)
-		(property "Reference" "C12"
+		(property "Reference" "C?"
 			(at 147.32 84.074 90)
 			(effects
@@
 					(unit 1)
 				)
+				(path "/f41306b9-7b2a-47ad-8a6e-226fbfa024ae/5235c0b2-ed00-4052-87b3-aafa4437d860/838d61aa-bfd3-43b0-96be-35c67846f33d"
+					(reference "C?")
+					(unit 1)
+				)
+				(path "/f41306b9-7b2a-47ad-8a6e-226fbfa024ae/5235c0b2-ed00-4052-87b3-aafa4437d860/fdd530e1-065e-4c92-a13d-ffa8fd694749"
+					(reference "C?")
+					(unit 1)
+				)
 			)
 		)
@@
 		(on_board yes)
 		(dnp no)
-		(property "Reference" "#PWR014"
+		(property "Reference" "#PWR?"
 			(at 133.35 127 0)
 			(effects
@@
 					(unit 1)
 				)
+				(path "/f41306b9-7b2a-47ad-8a6e-226fbfa024ae/5235c0b2-ed00-4052-87b3-aafa4437d860/838d61aa-bfd3-43b0-96be-35c67846f33d"
+					(reference "#PWR?")
+					(unit 1)
+				)
+				(path "/f41306b9-7b2a-47ad-8a6e-226fbfa024ae/5235c0b2-ed00-4052-87b3-aafa4437d860/fdd530e1-065e-4c92-a13d-ffa8fd694749"
+					(reference "#PWR?")
+					(unit 1)
+				)
 			)
 		)
@@
 		(on_board yes)
 		(dnp no)
-		(property "Reference" "#PWR011"
+		(property "Reference" "#PWR?"
 			(at 115.57 87.63 0)
 			(effects
@@
 					(unit 1)
 				)
+				(path "/f41306b9-7b2a-47ad-8a6e-226fbfa024ae/5235c0b2-ed00-4052-87b3-aafa4437d860/838d61aa-bfd3-43b0-96be-35c67846f33d"
+					(reference "#PWR?")
+					(unit 1)
+				)
+				(path "/f41306b9-7b2a-47ad-8a6e-226fbfa024ae/5235c0b2-ed00-4052-87b3-aafa4437d860/fdd530e1-065e-4c92-a13d-ffa8fd694749"
+					(reference "#PWR?")
+					(unit 1)
+				)
 			)
 		)
@@
 		(dnp no)
 		(fields_autoplaced yes)
-		(property "Reference" "R10"
+		(property "Reference" "R?"
 			(at 135.89 88.8999 0)
 			(effects
@@
 					(unit 1)
 				)
+				(path "/f41306b9-7b2a-47ad-8a6e-226fbfa024ae/5235c0b2-ed00-4052-87b3-aafa4437d860/838d61aa-bfd3-43b0-96be-35c67846f33d"
+					(reference "R?")
+					(unit 1)
+				)
+				(path "/f41306b9-7b2a-47ad-8a6e-226fbfa024ae/5235c0b2-ed00-4052-87b3-aafa4437d860/fdd530e1-065e-4c92-a13d-ffa8fd694749"
+					(reference "R?")
+					(unit 1)
+				)
 			)
 		)
@@
 		(dnp no)
 		(fields_autoplaced yes)
-		(property "Reference" "Q2"
+		(property "Reference" "Q?"
 			(at 135.89 107.9499 0)
 			(effects
@@
 					(unit 1)
 				)
+				(path "/f41306b9-7b2a-47ad-8a6e-226fbfa024ae/5235c0b2-ed00-4052-87b3-aafa4437d860/838d61aa-bfd3-43b0-96be-35c67846f33d"
+					(reference "Q?")
+					(unit 1)
+				)
+				(path "/f41306b9-7b2a-47ad-8a6e-226fbfa024ae/5235c0b2-ed00-4052-87b3-aafa4437d860/fdd530e1-065e-4c92-a13d-ffa8fd694749"
+					(reference "Q?")
+					(unit 1)
+				)
 			)
 		)
@@
 		(on_board yes)
 		(dnp no)
-		(property "Reference" "R9"
+		(property "Reference" "R?"
 			(at 153.67 87.884 0)
 			(effects
@@
 					(unit 1)
 				)
+				(path "/f41306b9-7b2a-47ad-8a6e-226fbfa024ae/5235c0b2-ed00-4052-87b3-aafa4437d860/838d61aa-bfd3-43b0-96be-35c67846f33d"
+					(reference "R?")
+					(unit 1)
+				)
+				(path "/f41306b9-7b2a-47ad-8a6e-226fbfa024ae/5235c0b2-ed00-4052-87b3-aafa4437d860/fdd530e1-065e-4c92-a13d-ffa8fd694749"
+					(reference "R?")
+					(unit 1)
+				)
 			)
 		)
@@
 		(on_board yes)
 		(dnp no)
-		(property "Reference" "#PWR012"
+		(property "Reference" "#PWR?"
 			(at 143.51 90.17 0)
 			(effects
@@
 					(unit 1)
 				)
+				(path "/f41306b9-7b2a-47ad-8a6e-226fbfa024ae/5235c0b2-ed00-4052-87b3-aafa4437d860/838d61aa-bfd3-43b0-96be-35c67846f33d"
+					(reference "#PWR?")
+					(unit 1)
+				)
+				(path "/f41306b9-7b2a-47ad-8a6e-226fbfa024ae/5235c0b2-ed00-4052-87b3-aafa4437d860/fdd530e1-065e-4c92-a13d-ffa8fd694749"
+					(reference "#PWR?")
+					(unit 1)
+				)
 			)
 		)
@@
 		(on_board yes)
 		(dnp no)
-		(property "Reference" "U5"
+		(property "Reference" "U?"
 			(at 139.7 94.234 0)
 			(effects
@@
 		)
 		(property "Value" "PC817"
-			(at 146.05 94.488 0)
+			(at 144.526 94.234 0)
 			(effects
 				(font
@@
 					(unit 1)
 				)
+				(path "/f41306b9-7b2a-47ad-8a6e-226fbfa024ae/5235c0b2-ed00-4052-87b3-aafa4437d860/838d61aa-bfd3-43b0-96be-35c67846f33d"
+					(reference "U?")
+					(unit 1)
+				)
+				(path "/f41306b9-7b2a-47ad-8a6e-226fbfa024ae/5235c0b2-ed00-4052-87b3-aafa4437d860/fdd530e1-065e-4c92-a13d-ffa8fd694749"
+					(reference "U?")
+					(unit 1)
+				)
