File: UV360/pir_sensors.kicad_sch (KiCad schematic)
At the start: 0 parts

Commit message: pir
copied from old
Parts:
- added C1: 0.1uf, Capacitor_THT:C_Disc_D3.8mm_W2.6mm_P2.50mm, symbol Device:C_Small
- added J1: PIR, TerminalBlock_Phoenix:TerminalBlock_Phoenix_MKDS-1,5-5-5.08_1x05_P5.08mm_Horizontal, symbol Connector:Screw_Terminal_01x05
Connections:
- new net 3.3V: C1.2, J1.2 (Pin_2)
- new net GND: C1.1, J1.1 (Pin_1)
- new net PIR_ISOLATOR/PIR: J1.3 (Pin_3)
- new net PIR_ISOLATOR1/PIR: J1.4 (Pin_4)
- new net PIR_ISOLATOR2/PIR: J1.5 (Pin_5)
Other:
- added sheet PIR_ISOLATOR (pir_isolator.kicad_sch)
- added sheet PIR_ISOLATOR1 (pir_isolator.kicad_sch)
- added sheet PIR_ISOLATOR2 (pir_isolator.kicad_sch)

Commit message: PIR
Other:
- sheet PIR_ISOLATOR ports: added +3.3V, +5V, GND-3.3V, GND-5V; removed none
- sheet PIR_ISOLATOR1 ports: added +3.3V, +5V, GND-3.3V, GND-5V; removed none
- sheet PIR_ISOLATOR2 ports: added +3.3V, +5V, GND-3.3V, GND-5V; removed none
